Commit message: Design & Policy Co-Optimisation Runner Updates
Problem
=======
1. Morphology Generation Methods hangs
2. Crash observed in `_reload_morphology` due to non-inference mode
   update of specific tensors
3. Incorrect Constructor Signature used for `UrdfConverterCfg`
4. Crash observed in `respawn_robots` to to None type `SpawnerCfg` of
   current articulation after first morphology update
5. URDF File not representative of Tron1
6. Incorrect name registered for Co-Optimisation Runner
7. Co-Optimisation Runner is set to run for 50000 steps, which is too
   much

Solution
========
1. Updated the name of the registered Co-Optimisation runner task in
   `tasks/locomotion/robots/__init__.py` in the package `exts/bipedal_locomotion`
2. Reduced the number of max_iterations to 15000 in
   `tasks/locomotion/agents/limx_rsl_rl_ppo_cfg.py` for `class
   SFCoptPPORunnerCfg` in the package `exts/bipedal_locomotion`
3. Updated URDF for Co-Optimisation Runner experiments at
   `assets/urdf/solefoot/base_robot.urdf` in the package `exts/bipedal_locomotion`
4. Converted `respawn_robots` from a method to class to persistently
   hold `rigid_props`, `articulation_props` and `activate_contact_sensors` in
   `co_optimisation/utils/respawn.py` in the package `co_optimisation`
5. Corrected Constructor Signature usage of `class UrdfConverterCfg` in
   `co_optimisation/runners/usd_generator.py`
6. Morphology generator was hanging due to the simulation not being
   flushed at stop, due to an internal private flag. Updating the flag
   manually fixes the issue
7. Added explicit `torch.inference_mode()` toggl before invocation of
   `_reload_morphology()` in
   `co_optimisation/runners/copt_on_policy_runner.py` in the package
   `co_optimisation`

Note
====
1. Added logs in the morphology update algorithm
2. Updated `lowest_terrain_camera_wrapper.py` to
   `highest_terrain_camera_wrapper.py` to track highest terrain walker
3. Updated imports in `scripts/rsl_rl/train.py` and
   `scripts/rsl_rl/play.py` to accomodate for update to
   `highest_terrain_camera_wrapper.py`
4. Added all assets needed by the URDF for experimentation

File: exts/bipedal_locomotion/bipedal_locomotion/assets/urdf/solefoot/base_robot.urdf (robot description, URDF)
Before this commit: robot SF_TRON1A, 10 links, 9 joints
Links:
- link abad_L_Link: geometry collision cylinder length=0.05 radius=0.05; visual cylinder length=0.05 radius=0.05
- link abad_R_Link: geometry collision cylinder length=0.05 radius=0.05; visual cylinder length=0.05 radius=0.05
- link ankle_L_Link: mass 0.620 -> 0.62; geometry collision mesh filename=file:///workspace/isaaclab/biped/exts/bipedal_locomotion/bi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 scale=1. 1. 1.; visual mesh filename=file:///workspace/isaaclab/biped/exts/bipedal_locomotion/bi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 scale=1. 1. 1.
- link ankle_R_Link: mass 0.620 -> 0.62; geometry collision mesh filename=file:///workspace/isaaclab/biped/exts/bipedal_locomotion/bi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 scale=1. 1. 1.; visual mesh filename=file:///workspace/isaaclab/biped/exts/bipedal_locomotion/bi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 scale=1. 1. 1.
- link base_Link: geometry collision box size=0.27 0.26 0.19; visual box size=0.27 0.26 0.19
- link hip_L_Link: mass 2.300 -> 2.3; geometry collision cylinder length=0.15 radius=0.035; visual cylinder length=0.15 radius=0.035
- link hip_R_Link: mass 2.300 -> 2.3; geometry collision cylinder length=0.15 radius=0.035; visual cylinder length=0.15 radius=0.035
- link knee_L_Link: mass 1.220 -> 1.22; geometry collision cylinder length=0.26 radius=0.02; visual cylinder length=0.26 radius=0.02
- link knee_R_Link: mass 1.220 -> 1.22; geometry collision cylinder length=0.26 radius=0.02; visual cylinder length=0.26 radius=0.02
- link limx_imu: mass 0.010 -> 0.01; geometry visual box size=0.015 0.015 0.004
Joints:
- joint abad_L_Joint: axis 1 0 0 -> 1. 0. 0.; limit lower=-0.3840 upper=1.3963 effort=40 velocity=23 -> lower=-0.38397 upper=1.3962599 effort=80. velocity=14.9999992; origin xyz=0.05556 0.105 -0.2602 rpy=0 0 0 -> xyz=0.05556 0.105 -0.2602  rpy=0. 0. 0.
- joint abad_R_Joint: axis 1 0 0 -> 1. 0. 0.; limit lower=-1.3963 upper=0.3840 effort=40 velocity=23 -> lower=-1.3962599 upper=0.38397 effort=80. velocity=14.9999992; origin xyz=0.05556 -0.105 -0.2602 rpy=0 0 0 -> xyz=0.05556 -0.105 -0.2602  rpy=0. 0. 0.
- joint ankle_L_Joint: axis 0 1 0 -> 0. 1. 0.; limit lower=-1.1519 upper=1.5708 effort=40 velocity=30 -> lower=-1.1519173 upper=1.5707963 effort=20. velocity=14.9999992; origin xyz=0.15 0 -0.25981 rpy=0 0 0 -> xyz=0.15 0. 0.25981 rpy=0. 0. 0.
- joint ankle_R_Joint: axis 0 1 0 -> 0. 1. 0.; limit lower=-1.1519 upper=1.5708 effort=40 velocity=30 -> lower=-1.1519173 upper=1.5707963 effort=20. velocity=14.9999992; origin xyz=0.15 0 -0.25981 rpy=0 0 0 -> xyz=0.15 0. -0.25981 rpy=3.1415927 0. 0. 
- joint hip_L_Joint: axis 0 1 0 -> 0. 1. 0.; limit lower=-1.0123 upper=1.3963 effort=60 velocity=20 -> lower=-1.0122909 upper=1.3962629 effort=80. velocity=14.9999992; origin xyz=-0.077 0.0205 0 rpy=0 0 0 -> xyz=-0.077 0.0205 0.  rpy=0. 0. 0.
- joint hip_R_Joint: axis 0 1 0 -> 0. 1. 0.; limit lower=-1.3963 upper=1.0123 effort=60 velocity=20 -> lower=-1.3962629 upper=1.0122909 effort=80. velocity=14.9999992; origin xyz=-0.077 -0.0205 0 rpy=0 0 0 -> xyz=-0.077 -0.0205 0.  rpy=3.1415927 0. 0. 
- joint knee_L_Joint: axis 0 1 0 -> 0. 1. 0.; limit lower=-0.8727 upper=1.3614 effort=60 velocity=14 -> lower=-0.872665 upper=1.3613569 effort=80. velocity=14.9999992; origin xyz=-0.15 -0.0205 -0.25981 rpy=0 0 0 -> xyz=-0.15 -0.0205 -0.25981 rpy=3.1415927 0. 0. 
- joint knee_R_Joint: axis 0 1 0 -> 0. 1. 0.; limit lower=-1.3614 upper=0.8727 effort=60 velocity=14 -> lower=-1.3613569 upper=0.872665 effort=80. velocity=14.9999992; origin xyz=-0.15 0.0205 -0.25981 rpy=0 0 0 -> xyz=-0.15 -0.0205 0.25981 rpy=3.1415927 0. 0. 
- joint limx_imu_joint: origin xyz=0 0 0 rpy=0 0 0 -> xyz=0. 0. 0. rpy=0. 0. 0.

Commit message: Base URDF for Co-Optimisation and Spawner Bug Fixes
Problem
=======
1. Joint Stiffness and Damping gains not added to spawned population
2. Crashes observed in spawned environments due to incorrect
   articulation references
3. Need to implement URDF Spawner and fix URDF for IsaacLab simulation

Solution
========
1. Added stiffness and damping paramter update in `class
   RandomDesignGenerator` in
   `co_optimisation/co_optimisation/runners/usd_generator.py`
2. Command and event manager were storing references to previously
   spawned articulation and need a reset of articulation at respawn
   implemented at `utils/respawn.py` in the package `co_optimisation`
3. Added `SOLEFOOT_CFG_URDF` and `SOLEFOOT_IDENTIFIED_CFG_URDF` in
   `assets/config/solefoot_cfg.py` and
   `assets/config/solefoot_identified_cfg.py` in the package `exts/bipedal_locomotion`
4. Removed self-collisions, added ankle joint and ensured tron 1 leg
   configuration and initial poses in
   `assets/urdf/solefoot/base_robot.urdf` in the package `exts/bipedal_locomotion`
5. Registered URDF spawner tasks in `tasks/locomotion/robots/__init__.py`

Note
====
1. Added inertia computation documentation at
   `assets/urdf/solefoot/base_robot.md` in the package `exts/bipedal_locomotion`

File: exts/bipedal_locomotion/bipedal_locomotion/assets/urdf/solefoot/base_robot.urdf (robot description, URDF)
Before this commit: robot SF_TRON1A, 10 links, 9 joints
Links:
- added link abad_L_actuator_Link, mass 0.95; collision cylinder length=0.0545 radius=0.0483; visual cylinder length=0.0545 radius=0.0483
- added link abad_R_actuator_Link, mass 0.95; collision cylinder length=0.0545 radius=0.0483; visual cylinder length=0.0545 radius=0.0483
- added link ankle_L_actuator_Link, mass 0.95; collision cylinder length=0.0545 radius=0.03; visual cylinder length=0.0545 radius=0.03
- added link ankle_R_actuator_Link, mass 0.95; collision cylinder length=0.0545 radius=0.03; visual cylinder length=0.0545 radius=0.03
- added link hip_L_thigh_Link, mass 1.5; collision box size=0.05 0.032 0.25; collision cylinder length=0.032 radius=0.0483
- added link hip_R_thigh_Link, mass 1.5; collision box size=0.05 0.032 0.25; collision cylinder length=0.032 radius=0.0483
- link abad_L_Link: geometry collision cylinder length=0.0545 radius=0.0483; visual cylinder length=0.0545 radius=0.0483
- link abad_R_Link: geometry collision cylinder length=0.0545 radius=0.0483; visual cylinder length=0.0545 radius=0.0483
- link ankle_L_Link: geometry collision box size=0.2 0.07 0.03; visual box size=0.2 0.07 0.03
- link ankle_R_Link: geometry collision box size=0.2 0.07 0.03; visual box size=0.2 0.07 0.03
- link base_Link: mass 9.585 -> 5; geometry collision box size=0.27 0.26 0.19; visual box size=0.27 0.26 0.19
- link hip_L_Link: mass 2.3 -> 0.95; geometry collision cylinder length=0.0545 radius=0.0483; visual cylinder length=0.0545 radius=0.0483
- link hip_R_Link: mass 2.3 -> 0.95; geometry collision cylinder length=0.0545 radius=0.0483; visual cylinder length=0.0545 radius=0.0483
- link knee_L_Link: geometry collision box size=0.025 0.032 0.3; visual box size=0.025 0.032 0.3
- link knee_R_Link: geometry collision box size=0.025 0.032 0.3; visual box size=0.025 0.032 0.3
Joints:
- added joint abad_L_fixed_joint: type fixed, parent base_Link, child abad_L_actuator_Link, origin xyz=0.08865 0.0817 -0.1875 rpy=0 0 0
- added joint abad_R_fixed_joint: type fixed, parent base_Link, child abad_R_actuator_Link, origin xyz=0.08865 -0.0817 -0.1875 rpy=0 0 0
- added joint ankle_L_actuator_Joint: type fixed, parent knee_L_Link, child ankle_L_actuator_Link, origin xyz=0.018 0 -0.34 rpy=0 0.6982 0
- added joint ankle_R_actuator_Joint: type fixed, parent knee_R_Link, child ankle_R_actuator_Link, origin xyz=0.018 0 -0.34 rpy=0 0.6982 0
- added joint hip_L_fixed_joint: type fixed, parent hip_L_Link, child hip_L_thigh_Link, origin xyz=0 0.08275 0 rpy=0 0.610865 0
- added joint hip_R_fixed_joint: type fixed, parent hip_R_Link, child hip_R_thigh_Link, origin xyz=0 -0.08275 0 rpy=0 0.610865 0
- joint abad_L_Joint: axis 1. 0. 0. -> 1 0 0; limit lower=-0.38397 upper=1.3962599 effort=80. velocity=14.9999992 -> lower=-0.38397 upper=1.39626 effort=80.0 velocity=15.0; origin xyz=0.05556 0.105 -0.2602  rpy=0. 0. 0. -> xyz=-0.0545 0 0 rpy=0 0 0; parent base_Link -> abad_L_actuator_Link
- joint abad_R_Joint: axis 1. 0. 0. -> -1 0 0; limit lower=-1.3962599 upper=0.38397 effort=80. velocity=14.9999992 -> lower=-0.38397 upper=1.39626 effort=80.0 velocity=15.0; origin xyz=0.05556 -0.105 -0.2602  rpy=0. 0. 0. -> xyz=-0.0545 0 0 rpy=0 0 0; parent base_Link -> abad_R_actuator_Link
- joint ankle_L_Joint: axis 0. 1. 0. -> 0 -1 0; limit lower=-1.1519173 upper=1.5707963 effort=20. velocity=14.9999992 -> lower=-0.79191730631626 upper=1.30899 effort=20 velocity=15; origin xyz=0.15 0. 0.25981 rpy=0. 0. 0. -> xyz=-0.025 0 -0.025 rpy=0 0 0; parent knee_L_Link -> ankle_L_actuator_Link
- joint ankle_R_Joint: axis 0. 1. 0. -> 0 -1 0; limit lower=-1.1519173 upper=1.5707963 effort=20. velocity=14.9999992 -> lower=-0.79191730631626 upper=1.30899 effort=20 velocity=15; origin xyz=0.15 0. -0.25981 rpy=3.1415927 0. 0.  -> xyz=-0.025 0 -0.025 rpy=0 0 0; parent knee_R_Link -> ankle_R_actuator_Link
- joint hip_L_Joint: axis 0. 1. 0. -> 0 1 0; limit lower=-1.0122909 upper=1.3962629 effort=80. velocity=14.9999992 -> lower=-1.012291 upper=1.396263 effort=80.0 velocity=15.0; origin xyz=-0.077 0.0205 0.  rpy=0. 0. 0. -> xyz=-0.0683 -0.03050 0 rpy=0 0 0
- joint hip_R_Joint: axis 0. 1. 0. -> 0 -1 0; limit lower=-1.3962629 upper=1.0122909 effort=80. velocity=14.9999992 -> lower=-1.396263 upper=1.012291 effort=80.0 velocity=15.0; origin xyz=-0.077 -0.0205 0.  rpy=3.1415927 0. 0.  -> xyz=-0.0683 0.03050 0 rpy=0 0 0
- joint knee_L_Joint: axis 0. 1. 0. -> 0 -1 0; limit lower=-0.872665 upper=1.3613569 effort=80. velocity=14.9999992 -> lower=-0.872665 upper=1.361357 effort=80 velocity=15; origin xyz=-0.15 -0.0205 -0.25981 rpy=3.1415927 0. 0.  -> xyz=0 -0.04325 -0.35 rpy=0 -1.3090 0; parent hip_L_Link -> hip_L_thigh_Link
- joint knee_R_Joint: axis 0. 1. 0. -> 0 -1 0; limit lower=-1.3613569 upper=0.872665 effort=80. velocity=14.9999992 -> lower=-1.21357 upper=1.172665 effort=80 velocity=15; origin xyz=-0.15 -0.0205 0.25981 rpy=3.1415927 0. 0.  -> xyz=0 0.04325 -0.35 rpy=0 -1.3090 0; parent hip_R_Link -> hip_R_thigh_Link
- joint limx_imu_joint: origin xyz=0. 0. 0. rpy=0. 0. 0. -> xyz=0 0 0 rpy=0 0 0

Commit message: URDF update for co-design optimisation integration
Problem
=======
1. Number of joint reducing due to fixed joint merging leading to crash
   at the start of the training due to missing hip flexion and extension
   and hip abduction and adduction links
2. `SOLEFOOT_IDENTIFIED_MULTIUSD_CFG` is not functional and is needed
   for initialisation of the environment with appropriate individual
   indexing within the environment for appropriate design
   optimisation based on fitness from PPO training
3. Need to update joint topology and ensure placement for joints for
   easy design updates during training

Solution
========
1. Set `merge_fixed_joints` to False to ensure no fixed joints are
   merged in the final articulation used in Isaac Lab in
   `assets/config/solefoot_identified_cfg.py` and
   `assets/config/solefoot_cfg.py` in the package `exts/bipedal_locomotion`
2. Using `UrdfConverterCfg` and `UrdfConverter` to convert URDF files
   into multiple USDs to simulate individuals within the simulation
   which are to be later updated to create a varying population in
   `assets/config/solefoot_identified_cfg.py` in the package
   `exts/bipedal_locomotion`
3. Updated `assets/urdf/solefoot/base_robot.urdf` to ensure joints in
   such a way that increasing the size of a link means increasing the
   offset between parent and child frames in the joints by the same
   amount as that of the link length change. This is done to ensure the
   final linkages created after design updates are valid without any
   dangling or overshooting links. Updated moment of inertia computation
   for `assets/urdf/solefoot/base_robot.md`. All changes are in the
   package `exts/bipedal_locomotion`.

Note
====

File: exts/bipedal_locomotion/bipedal_locomotion/assets/urdf/solefoot/base_robot.urdf (robot description, URDF)
Before this commit: robot SF_TRON1, 16 links, 15 joints
Links:
- removed link abad_L_Link
- removed link abad_R_Link
- added link hip_L_actuator_Link, mass 1.469; collision cylinder length=0.0545 radius=0.0483; visual cylinder length=0.0545 radius=0.0483
- added link hip_R_actuator_Link, mass 1.469; collision cylinder length=0.0545 radius=0.0483; visual cylinder length=0.0545 radius=0.0483
- added link knee_L_actuator_Link, mass 0.95; collision cylinder length=0.0545 radius=0.0483; visual cylinder length=0.0545 radius=0.0483
- added link knee_R_actuator_Link, mass 0.95; collision cylinder length=0.0545 radius=0.0483; visual cylinder length=0.0545 radius=0.0483
- link hip_L_Link: mass 0.95 -> 0.5; geometry collision cylinder length=0.032 radius=0.0483; visual cylinder length=0.032 radius=0.0483
- link hip_L_thigh_Link: geometry collision box size=0.05 0.032 0.25; visual box size=0.05 0.032 0.25
- link hip_R_Link: mass 0.95 -> 0.5; geometry collision cylinder length=0.032 radius=0.0483; visual cylinder length=0.032 radius=0.0483
- link hip_R_thigh_Link: geometry collision box size=0.05 0.032 0.25; visual box size=0.05 0.032 0.25
Joints:
- added joint knee_L_actuator_joint: type fixed, parent hip_L_Link, child knee_L_actuator_Link, origin xyz=0 0.032 0 rpy=0 0 0
- added joint knee_R_actuator_joint: type fixed, parent hip_R_Link, child knee_R_actuator_Link, origin xyz=0 -0.032 0 rpy=0 0 0
- joint abad_L_Joint: child abad_L_Link -> hip_L_actuator_Link; origin xyz=-0.0545 0 0 rpy=0 0 0 -> xyz=-0.0683 0 0 rpy=0 0 0
- joint abad_L_fixed_joint: origin xyz=0.08865 0.0817 -0.1875 rpy=0 0 0 -> xyz=0.06 0.0817 -0.1875 rpy=0 0 0
- joint abad_R_Joint: child abad_R_Link -> hip_R_actuator_Link; origin xyz=-0.0545 0 0 rpy=0 0 0 -> xyz=-0.0683 0 0 rpy=0 0 0
- joint abad_R_fixed_joint: origin xyz=0.08865 -0.0817 -0.1875 rpy=0 0 0 -> xyz=0.06 -0.0817 -0.1875 rpy=0 0 0
- joint ankle_L_actuator_Joint: origin xyz=0.018 0 -0.34 rpy=0 0.6982 0 -> xyz=0.018 0 -0.35 rpy=0 0.6982 0
- joint ankle_R_actuator_Joint: origin xyz=0.018 0 -0.34 rpy=0 0.6982 0 -> xyz=0.018 0 -0.35 rpy=0 0.6982 0
- joint hip_L_Joint: origin xyz=-0.0683 -0.03050 0 rpy=0 0 0 -> xyz=0 -0.00775 0 rpy=0 0.610865 0; parent abad_L_Link -> hip_L_actuator_Link
- joint hip_L_fixed_joint: origin xyz=0 0.08275 0 rpy=0 0.610865 0 -> xyz=0 0.016 -0.0483 rpy=0 0 0
- joint hip_R_Joint: origin xyz=-0.0683 0.03050 0 rpy=0 0 0 -> xyz=0 0.00775 0 rpy=0 0.610865 0; parent abad_R_Link -> hip_R_actuator_Link
- joint hip_R_fixed_joint: origin xyz=0 -0.08275 0 rpy=0 0.610865 0 -> xyz=0 -0.016 -0.0483 rpy=0 0 0
- joint knee_L_Joint: origin xyz=0 -0.04325 -0.35 rpy=0 -1.3090 0 -> xyz=0 0 -0.3 rpy=0 -1.3090 0
- joint knee_R_Joint: origin xyz=0 0.04325 -0.35 rpy=0 -1.3090 0 -> xyz=0 0 -0.3 rpy=0 -1.3090 0
